Commit message: delete .gazebo.xacro (not used)

File: echo_bot_common/echo_bot_description/robots/echo_bot.urdf.xacro (robot description, xacro)
@@ -5,4 +5,6 @@
   <xacro:include filename="$(find echo_bot_description)/urdf/leg/echo_bot_leg.urdf.xacro"/>
   <xacro:include filename="$(find echo_bot_description)/urdf/wheel/echo_bot_wheel.urdf.xacro"/>
+  <xacro:include filename="$(find echo_bot_description)/urdf/sensors/lidar/lidar.urdf.xacro"/>
+  <xacro:include filename="$(find echo_bot_description)/urdf/sensors/imu/imu.urdf.xacro"/>
   <!-- == echo_bot base == -->
   <link name="base_link"/>
@@ -13,8 +15,4 @@
     <child link="torso_link"/>
   </joint>
-  <!-- <link name="world"/>
-  <xacro:torso_v0 parent="world">
-  <origin xyz="0 0 0.20"/>
-  </xacro:torso_v0> -->
   <!-- <link name="base_footprint"/>
   <joint name="base_link_to_base_footprint_joint" type="fixed">
@@ -41,24 +39,10 @@
     <axis xyz="0 0 1"/>
   </xacro:wheel_v0>
-  <!-- == Sensor == -->
-  <!-- == Gazebo == -->
-  <gazebo>
-    <plugin name="gazebo_ros_control" filename="libgazebo_ros_control.so">
-      <robotNamespace>echo_bot</robotNamespace>
-      <robotSimType>gazebo_ros_control/DefaultRobotHWSim</robotSimType>
-      <legacyModeNS>true</legacyModeNS>
-    </plugin>
-  </gazebo>
-  <plugin name="joint_state_publisher" filename="libgazebo_ros_joint_state_publisher.so">
-    <robotNamespace>echo_bot</robotNamespace>
-    <jointName>torso_to_upper_lleg, torso_to_upper_rleg, upper_lleg_to_lower_lleg, upper_rleg_to_lower_rleg, lower_lleg_to_upper_side_lleg, lower_rleg_to_upper_side_rleg, lower_lleg_to_wheel_l, lower_rleg_to_wheel_r</jointName>
-  </plugin>
-  <!-- Base -->
-  <xacro:torso_gazebo_v0/>
-  <!-- leg -->
-  <xacro:leg_gazebo_v0 prefix="l"/>
-  <xacro:leg_gazebo_v0 prefix="r"/>
-  <!-- Wheel -->
-  <xacro:wheel_gazebo_v0 prefix="l"/>
-  <xacro:wheel_gazebo_v0 prefix="r"/>
+  <!-- == Sensors == -->
+  <xacro:lidar_v0 parent="torso_link">
+    <origin xyz="0 0 0.11" rpy="0 0 0"/>
+  </xacro:lidar_v0>
+  <xacro:imu_v0 parent="torso_link">
+    <origin xyz="0 0 0" rpy="0 0 0"/>
+  </xacro:imu_v0>
 </robot>

File: echo_bot_common/echo_bot_description/urdf/leg/echo_bot_leg.urdf.xacro (robot description, xacro)
@@ -2,5 +2,4 @@
 <robot xmlns:xacro="http://ros.org/wiki/xacro">
   <xacro:include filename="$(find echo_bot_description)/urdf/leg/echo_bot_leg.transmission.xacro"/>
-  <xacro:include filename="$(find echo_bot_description)/urdf/leg/echo_bot_leg.gazebo.xacro"/>
   <xacro:macro name="leg_v0" params="parent prefix *joint_origin">
     <!-- Link -->

File: echo_bot_common/echo_bot_description/urdf/torso/echo_bot_torso.urdf.xacro (robot description, xacro)
@@ -1,5 +1,4 @@
 <?xml version="1.0"?>
 <robot xmlns:xacro="http://ros.org/wiki/xacro">
-  <xacro:include filename="$(find echo_bot_description)/urdf/torso/echo_bot_torso.gazebo.xacro"/>
   <xacro:macro name="torso_v0">
     <link name="torso_link">

File: echo_bot_common/echo_bot_description/urdf/wheel/echo_bot_wheel.urdf.xacro (robot description, xacro)
@@ -2,5 +2,4 @@
 <robot xmlns:xacro="http://ros.org/wiki/xacro">
   <xacro:include filename="$(find echo_bot_description)/urdf/wheel/echo_bot_wheel.transmission.xacro"/>
-  <xacro:include filename="$(find echo_bot_description)/urdf/wheel/echo_bot_wheel.gazebo.xacro"/>
   <property name="wheel_radius" value="0.029"/>
   <property name="wheel_length" value="0.012"/>
