Commit message: update models

File: echo_bot_common/echo_bot_description/urdf/leg/echo_bot_leg.urdf.xacro (robot description, xacro)
@@ -8,5 +8,5 @@
         <origin xyz="0 0 0" rpy="0 0 0"/>
         <geometry>
-          <mesh filename="package://echo_bot_description/meshes/DAE/upper_leg.dae"/>
+          <mesh filename="package://echo_bot_description/meshes/DAE/upper_${prefix}leg.dae"/>
         </geometry>
       </visual>
@@ -14,5 +14,5 @@
         <origin xyz="0 0 0" rpy="0 0 0"/>
         <geometry>
-          <mesh filename="package://echo_bot_description/meshes/STL/upper_leg.stl"/>
+          <mesh filename="package://echo_bot_description/meshes/STL/upper_${prefix}leg.stl"/>
         </geometry>
       </collision>
@@ -57,5 +57,5 @@
         <material name="leg_color_0"/>
         <geometry>
-          <mesh filename="package://echo_bot_description/meshes/DAE/upper_side_leg.dae"/>
+          <mesh filename="package://echo_bot_description/meshes/DAE/upper_side_${prefix}leg.dae"/>
         </geometry>
       </visual>
@@ -63,5 +63,5 @@
         <origin xyz="0 0 0" rpy="0 0 0"/>
         <geometry>
-          <mesh filename="package://echo_bot_description/meshes/STL/upper_side_leg.stl"/>
+          <mesh filename="package://echo_bot_description/meshes/STL/upper_side_${prefix}leg.stl"/>
         </geometry>
       </collision>

File: echo_bot_common/echo_bot_description/urdf/wheel/echo_bot_wheel.urdf.xacro (robot description, xacro)
@@ -15,5 +15,5 @@
       <visual>
         <geometry>
-          <mesh filename="package://echo_bot_description/meshes/DAE/tyre.dae"/>
+          <mesh filename="package://echo_bot_description/meshes/DAE/wheel.dae"/>
         </geometry>
       </visual>
@@ -23,5 +23,5 @@
         <geometry>
           <!-- <cylinder radius="${wheel_radius}" length="${wheel_length}"/> -->
-          <mesh filename="package://echo_bot_description/meshes/STL/tyre.stl"/>
+          <mesh filename="package://echo_bot_description/meshes/STL/wheel.stl"/>
         </geometry>
       </collision>

Commit message: change parameter

File: echo_bot_common/echo_bot_description/urdf/leg/echo_bot_leg.urdf.xacro (robot description, xacro)
@@ -73,5 +73,5 @@
                   iyz="0.0"
                   izz="0.000314"/>
-        <mass value="0.5"/>
+        <mass value="0.017"/>
         <origin xyz="0.05 0 0" rpy="0 0 0"/>
       </inertial>

File: echo_bot_common/echo_bot_description/urdf/torso/echo_bot_torso.urdf.xacro (robot description, xacro)
@@ -16,12 +16,12 @@
       </collision>
       <inertial>
-        <inertia  ixx="0.006594"
-                  ixy="0.0"
-                  ixz="0.000999"
-                  iyy="0.007405"
-                  iyz="0.0"
-                  izz="0.010608"/>
-        <mass value="2.915"/>
-        <origin xyz="0.025 0 0.053" rpy="0 0 0"/>
+        <inertia  ixx="0.0028602"
+                  ixy="-0.0000824"
+                  ixz="0.0004955"
+                  iyy="0.0038656"
+                  iyz="-0.0000108"
+                  izz="0.0042401"/>
+        <mass value="1.23"/>
+        <origin xyz="0.006457 0 0.044346" rpy="0 0 0"/>
       </inertial>
     </link>
